File: Hardware/Mosfet Rpi Hat.sch (KiCad schematic (older format))
At the start: 6 parts

Commit message: added raspberry pi librarie
Just librarie (no footprint yet)
Connections:
- net GPIO: no longer R?.2
- new net PWM0: R?.2
Changed lines of the file:
@@
 GPIO
 Text GLabel 1250 1700 0    60   Input ~ 0
-GPIO
+PWM0
 $Comp
 L LTV-356T U?
